Commit message: robot moves, change configurations but problem on visualization

File: ur5e_2fg7/urdf/ur5e_2fg7_description_only.urdf.xacro (robot description, xacro)
@@ -14,6 +14,5 @@
     use_fake_hardware="true"
     fake_sensor_commands="false"
-    initial_positions="${dict(shoulder_pan_joint=0.0,shoulder_lift_joint=-1.57,elbow_joint=1.57,wrist_1_joint=-1.57,wrist_2_joint=-1.57,wrist_3_joint=0.0)}">
-    <origin xyz="0 0 0" rpy="0 0 0"/>
+    initial_positions="${dict(shoulder_pan_joint=-1.55334,shoulder_lift_joint=-1.97222,elbow_joint=1.88496,wrist_1_joint=-1.48353,wrist_2_joint=-1.5708,wrist_3_joint=-1.55334)}">    <origin xyz="0 0 0" rpy="0 0 0"/>
   </xacro:ur_robot>
   <xacro:onrobot_2fg7 parent="tool0" prefix="gripper_">

File: ur5e_2fg7_moveit_config/config/ur5e_con_2fg7.ros2_control.xacro (robot description, xacro)
@@ -5,11 +5,12 @@
         <ros2_control name="${name}" type="system">
             <hardware>
-                <!-- By default, set up controllers for simulation. This won't work on real hardware -->
+                <!-- Fake hardware for MoveIt/RViz simulation -->
                 <plugin>mock_components/GenericSystem</plugin>
             </hardware>
+            <!-- UR5e arm joints -->
             <joint name="shoulder_pan_joint">
                 <command_interface name="position"/>
                 <state_interface name="position">
-                  <param name="initial_value">${initial_positions['shoulder_pan_joint']}</param>
+                    <param name="initial_value">${initial_positions['shoulder_pan_joint']}</param>
                 </state_interface>
                 <state_interface name="velocity"/>
@@ -18,5 +19,5 @@
                 <command_interface name="position"/>
                 <state_interface name="position">
-                  <param name="initial_value">${initial_positions['shoulder_lift_joint']}</param>
+                    <param name="initial_value">${initial_positions['shoulder_lift_joint']}</param>
                 </state_interface>
                 <state_interface name="velocity"/>
@@ -25,5 +26,5 @@
                 <command_interface name="position"/>
                 <state_interface name="position">
-                  <param name="initial_value">${initial_positions['elbow_joint']}</param>
+                    <param name="initial_value">${initial_positions['elbow_joint']}</param>
                 </state_interface>
                 <state_interface name="velocity"/>
@@ -32,5 +33,5 @@
                 <command_interface name="position"/>
                 <state_interface name="position">
-                  <param name="initial_value">${initial_positions['wrist_1_joint']}</param>
+                    <param name="initial_value">${initial_positions['wrist_1_joint']}</param>
                 </state_interface>
                 <state_interface name="velocity"/>
@@ -39,5 +40,5 @@
                 <command_interface name="position"/>
                 <state_interface name="position">
-                  <param name="initial_value">${initial_positions['wrist_2_joint']}</param>
+                    <param name="initial_value">${initial_positions['wrist_2_joint']}</param>
                 </state_interface>
                 <state_interface name="velocity"/>
@@ -46,5 +47,22 @@
                 <command_interface name="position"/>
                 <state_interface name="position">
-                  <param name="initial_value">${initial_positions['wrist_3_joint']}</param>
+                    <param name="initial_value">${initial_positions['wrist_3_joint']}</param>
+                </state_interface>
+                <state_interface name="velocity"/>
+            </joint>
+            <!-- 2FG7 gripper joints.
+                 These are needed so joint_state_broadcaster publishes gripper states
+                 and robot_state_publisher can compute the finger transforms. -->
+            <joint name="gripper_gripper_joint">
+                <command_interface name="position"/>
+                <state_interface name="position">
+                    <param name="initial_value">${initial_positions['gripper_gripper_joint']}</param>
+                </state_interface>
+                <state_interface name="velocity"/>
+            </joint>
+            <joint name="gripper_right_finger_joint">
+                <command_interface name="position"/>
+                <state_interface name="position">
+                    <param name="initial_value">${initial_positions['gripper_right_finger_joint']}</param>
                 </state_interface>
                 <state_interface name="velocity"/>

File: ur5e_2fg7_moveit_config/config/ur5e_con_2fg7.urdf.xacro (robot description, xacro)
@@ -1,11 +1,11 @@
 <?xml version="1.0"?>
 <robot xmlns:xacro="http://www.ros.org/wiki/xacro" name="ur5e_con_2fg7">
-    <!--<xacro:arg name="initial_positions_file" default="initial_positions.yaml" /> -->
-    <!-- Robot description only: UR5e + 2FG7, without real UR hardware interface -->
+    <xacro:arg
+        name="initial_positions_file"
+        default="$(find ur5e_2fg7_moveit_config)/config/initial_positions.yaml" />
     <xacro:include filename="$(find ur5e_2fg7)/urdf/ur5e_2fg7_description_only.urdf.xacro" />
-    <!-- Fake ros2_control system for MoveIt/RViz simulation -->
-    <!--<xacro:include filename="$(find ur5e_2fg7_moveit_config)/config/ur5e_con_2fg7.ros2_control.xacro" />
+    <xacro:include filename="$(find ur5e_2fg7_moveit_config)/config/ur5e_con_2fg7.ros2_control.xacro" />
     <xacro:ur5e_con_2fg7_ros2_control
         name="FakeSystem"
-        initial_positions_file="$(arg initial_positions_file)" /> -->
+        initial_positions_file="$(arg initial_positions_file)" />
 </robot>

Commit message: motion from start to table

File: ur5e_2fg7/urdf/ur5e_2fg7_description_only.urdf.xacro (robot description, xacro)
@@ -14,5 +14,5 @@
     use_fake_hardware="true"
     fake_sensor_commands="false"
-    initial_positions="${dict(shoulder_pan_joint=-1.55334,shoulder_lift_joint=-1.97222,elbow_joint=1.88496,wrist_1_joint=-1.48353,wrist_2_joint=-1.5708,wrist_3_joint=-1.55334)}">    <origin xyz="0 0 0" rpy="0 0 0"/>
+    initial_positions="${dict(shoulder_pan_joint=0.0,shoulder_lift_joint=-1.5708,elbow_joint=0.0,wrist_1_joint=-1.5708,wrist_2_joint=0.0,wrist_3_joint=0.0)}">    <origin xyz="0 0 0" rpy="0 0 0"/>
   </xacro:ur_robot>
   <xacro:onrobot_2fg7 parent="tool0" prefix="gripper_">
